File: hardware/clockInterface.sch (KiCad schematic (older format))
At the start: 15 parts, among them P301 CLOCK1, P302 CLOCK2, SW301 SW_PUSH, SW302 SW_PUSH, SW303 SW_PUSH

Commit message: Opened schematic and pcb with kicad 5.1.5...
...to update library table
Parts:
- D301, D302, D303, D304, D305: symbol LED -> wfred_loconet_clock-rescue:LED
- P301, P302: symbol CONN_2 -> wfred_loconet_clock-rescue:CONN_2
- R301, R302, R303, R304, R305: symbol R -> wfred_loconet_clock-rescue:R
- SW301, SW302, SW303: symbol SW_PUSH -> wfred_loconet_clock-rescue:SW_PUSH
Changed lines of the file:
@@
-EESchema Schematic File Version 2
-LIBS:wfred_loconet_clock-rescue
-LIBS:power
-LIBS:device
-LIBS:transistors
-LIBS:conn
-LIBS:linear
-LIBS:regul
-LIBS:74xx
-LIBS:cmos4000
-LIBS:adc-dac
-LIBS:memory
-LIBS:xilinx
-LIBS:microcontrollers
-LIBS:dsp
-LIBS:microchip
-LIBS:analog_switches
-LIBS:motorola
-LIBS:texas
-LIBS:intel
-LIBS:audio
-LIBS:interface
-LIBS:digital-audio
-LIBS:philips
-LIBS:display
-LIBS:cypress
-LIBS:siliconi
-LIBS:opto
-LIBS:atmel
-LIBS:contrib
-LIBS:valves
-LIBS:my_devices
-LIBS:ESP8266
-LIBS:wfred_loconet_clock-cache
-EELAYER 25 0
+EESchema Schematic File Version 4
+EELAYER 30 0
 EELAYER END
 $Descr A4 11693 8268
@@
 CLOCK2
 $Comp
-L R R301
+L wfred_loconet_clock-rescue:R R301
 U 1 1 5A1291DD
 P 4450 2700
@@
 $EndComp
 $Comp
-L R R302
+L wfred_loconet_clock-rescue:R R302
 U 1 1 5A12924F
 P 4450 3500
@@
 $EndComp
 $Comp
-L LED D301
+L wfred_loconet_clock-rescue:LED D301
 U 1 1 5A12928F
 P 5000 3100
@@
 $EndComp
 $Comp
-L LED D302
+L wfred_loconet_clock-rescue:LED D302
 U 1 1 5A129325
 P 5300 3100
@@
 $EndComp
 $Comp
-L CONN_2 P301
+L wfred_loconet_clock-rescue:CONN_2 P301
 U 1 1 5A12938D
 P 6150 3100
@@
 	3900 2700 4200 2700
 Wire Wire Line
-	4700 2700 5600 2700
+	4700 2700 5000 2700
 Wire Wire Line
 	5600 2700 5600 3000
@@
 	3900 3500 4200 3500
 Wire Wire Line
-	4700 3500 5600 3500
+	4700 3500 5000 3500
 Wire Wire Line
 	5600 3500 5600 3200
@@
 Connection ~ 5000 3500
 $Comp
-L GND #PWR020
+L wfred_loconet_clock-rescue:GND #PWR020
 U 1 1 5A15360C
 P 5400 6900
@@
 	4400 4500 3900 4500
 $Comp
-L SW_PUSH SW301
+L wfred_loconet_clock-rescue:SW_PUSH SW301
 U 1 1 5C82A486
 P 4700 4500
@@
 $EndComp
 $Comp
-L LED D303
+L wfred_loconet_clock-rescue:LED D303
 U 1 1 5C82A97E
 P 6900 2700
@@
 $EndComp
 $Comp
-L R R303
+L wfred_loconet_clock-rescue:R R303
 U 1 1 5C82AAA2
 P 6900 3450
@@
 $EndComp
 $Comp
-L VCC #PWR021
+L wfred_loconet_clock-rescue:VCC #PWR021
 U 1 1 5C82ABFF
 P 6900 2200
@@
 	4400 4900 3900 4900
 $Comp
-L SW_PUSH SW302
+L wfred_loconet_clock-rescue:SW_PUSH SW302
 U 1 1 5CA9E853
 P 4700 4900
@@
 	4400 5300 3900 5300
 $Comp
-L SW_PUSH SW303
+L wfred_loconet_clock-rescue:SW_PUSH SW303
 U 1 1 5CA9E95A
 P 4700 5300
@@
 CLOCK4
 $Comp
-L R R304
+L wfred_loconet_clock-rescue:R R304
 U 1 1 5D44BDE6
 P 4450 1700
@@
 $EndComp
 $Comp
-L R R305
+L wfred_loconet_clock-rescue:R R305
 U 1 1 5D44BDED
 P 4450 2500
@@
 $EndComp
 $Comp
-L LED D304
+L wfred_loconet_clock-rescue:LED D304
 U 1 1 5D44BDF4
 P 5000 2100
@@
 $EndComp
 $Comp
-L LED D305
+L wfred_loconet_clock-rescue:LED D305
 U 1 1 5D44BDFB
 P 5300 2100
@@
 $EndComp
 $Comp
-L CONN_2 P302
+L wfred_loconet_clock-rescue:CONN_2 P302
 U 1 1 5D44BE02
 P 6150 2100
@@
 	3900 1700 4200 1700
 Wire Wire Line
-	4700 1700 5600 1700
+	4700 1700 5000 1700
 Wire Wire Line
 	5600 1700 5600 2000
@@
 	3900 2500 4200 2500
 Wire Wire Line
-	4700 2500 5600 2500
+	4700 2500 5000 2500
 Wire Wire Line
 	5600 2500 5600 2200
@@
 Connection ~ 5000 2500
 Wire Wire Line
-	5400 4500 5400 6900
+	5400 4500 5400 4900
+Wire Wire Line
+	5300 2700 5600 2700
+Wire Wire Line
+	5000 2700 5300 2700
+Wire Wire Line
+	5300 3500 5600 3500
+Wire Wire Line
+	5000 3500 5300 3500
+Wire Wire Line
+	5400 4900 5400 5300
+Wire Wire Line
+	5400 5300 5400 6900
+Wire Wire Line
+	5300 1700 5600 1700
+Wire Wire Line
+	5000 1700 5300 1700
+Wire Wire Line
+	5300 2500 5600 2500
+Wire Wire Line
+	5000 2500 5300 2500
 $EndSCHEMATC
