File: hardware/clockInterface.sch (KiCad schematic (older format))
At the start: 9 parts, among them P501 CLOCK, SW501 SWITCH_INV, SW502 SWITCH_INV, SW503 SWITCH_INV, SW504 SWITCH_INV

Commit message: Fixed up wfred_loconet_clock PCB...
...just in case someone actually wants to use it...
Parts:
- D501, D502: symbol LED -> wfred_loconet_clock-rescue:LED
- P501: symbol CONN_2 -> wfred_loconet_clock-rescue:CONN_2
- R501, R502: symbol R -> wfred_loconet_clock-rescue:R
- SW501, SW502, SW503, SW504: symbol SWITCH_INV -> wfred_loconet_clock-rescue:SWITCH_INV
Changed lines of the file:
@@
-EESchema Schematic File Version 2
-LIBS:power
-LIBS:device
-LIBS:transistors
-LIBS:conn
-LIBS:linear
-LIBS:regul
-LIBS:74xx
-LIBS:cmos4000
-LIBS:adc-dac
-LIBS:memory
-LIBS:xilinx
-LIBS:microcontrollers
-LIBS:dsp
-LIBS:microchip
-LIBS:analog_switches
-LIBS:motorola
-LIBS:texas
-LIBS:intel
-LIBS:audio
-LIBS:interface
-LIBS:digital-audio
-LIBS:philips
-LIBS:display
-LIBS:cypress
-LIBS:siliconi
-LIBS:opto
-LIBS:atmel
-LIBS:contrib
-LIBS:valves
-LIBS:my_devices
-LIBS:ESP8266
-LIBS:wfred_loconet_clock-cache
-EELAYER 25 0
+EESchema Schematic File Version 4
+EELAYER 30 0
 EELAYER END
 $Descr A4 11693 8268
@@
 CLOCK2
 $Comp
-L R R501
+L wfred_loconet_clock-rescue:R R501
 U 1 1 5A1291DD
 P 4450 2700
@@
 $EndComp
 $Comp
-L R R502
+L wfred_loconet_clock-rescue:R R502
 U 1 1 5A12924F
 P 4450 3500
@@
 $EndComp
 $Comp
-L LED D501
+L wfred_loconet_clock-rescue:LED D501
 U 1 1 5A12928F
 P 5000 3100
@@
 $EndComp
 $Comp
-L LED D502
+L wfred_loconet_clock-rescue:LED D502
 U 1 1 5A129325
 P 5300 3100
@@
 $EndComp
 $Comp
-L CONN_2 P501
+L wfred_loconet_clock-rescue:CONN_2 P501
 U 1 1 5A12938D
 P 6150 3100
@@
 	3900 2700 4200 2700
 Wire Wire Line
-	4700 2700 5600 2700
+	4700 2700 5000 2700
 Wire Wire Line
 	5600 2700 5600 3000
@@
 	3900 3500 4200 3500
 Wire Wire Line
-	4700 3500 5600 3500
+	4700 3500 5000 3500
 Wire Wire Line
 	5600 3500 5600 3200
@@
 Connection ~ 5000 3500
 $Comp
-L SWITCH_INV SW501
+L wfred_loconet_clock-rescue:SWITCH_INV SW501
 U 1 1 5A15342E
 P 4500 4100
@@
 $EndComp
 $Comp
-L SWITCH_INV SW502
+L wfred_loconet_clock-rescue:SWITCH_INV SW502
 U 1 1 5A15348B
 P 4500 4600
@@
 $EndComp
 $Comp
-L SWITCH_INV SW503
+L wfred_loconet_clock-rescue:SWITCH_INV SW503
 U 1 1 5A153526
 P 4500 5100
@@
 $EndComp
 $Comp
-L SWITCH_INV SW504
+L wfred_loconet_clock-rescue:SWITCH_INV SW504
 U 1 1 5A1535A1
 P 4500 5600
@@
 $EndComp
 $Comp
-L GND #PWR045
+L wfred_loconet_clock-rescue:GND #PWR045
 U 1 1 5A15360C
 P 3800 6100
@@
 $EndComp
 $Comp
-L GND #PWR046
+L wfred_loconet_clock-rescue:GND #PWR046
 U 1 1 5A15363B
 P 5200 6100
@@
 $EndComp
 Wire Wire Line
-	5200 6100 5200 4000
+	5200 6100 5200 5500
 Wire Wire Line
 	5200 4000 5000 4000
@@
 Connection ~ 5200 5500
 Wire Wire Line
-	3800 4100 3800 6100
+	3800 4100 3800 4600
 Wire Wire Line
 	3800 5600 4000 5600
@@
 Wire Wire Line
 	5000 5700 5350 5700
+Wire Wire Line
+	5300 2700 5600 2700
+Wire Wire Line
+	5000 2700 5300 2700
+Wire Wire Line
+	5300 3500 5600 3500
+Wire Wire Line
+	5000 3500 5300 3500
+Wire Wire Line
+	5200 4500 5200 4000
+Wire Wire Line
+	5200 5000 5200 4500
+Wire Wire Line
+	5200 5500 5200 5000
+Wire Wire Line
+	3800 5600 3800 6100
+Wire Wire Line
+	3800 5100 3800 5600
+Wire Wire Line
+	3800 4600 3800 5100
 $EndSCHEMATC
