File: hardware/loconet-interface.sch (KiCad schematic (older format))
At the start: 24 parts, among them J301 Molex 95501-6669, K301 TERMINATION, Q301 BC817-40, Q302 BC817-40, Q303 BC817-40, U301 TC1240

Commit message: Fixed up wfred_loconet_clock PCB...
...just in case someone actually wants to use it...
Parts:
- C301, C302, C303, C304, C305: symbol C -> wfred_loconet_clock-rescue:C
- D301, D302, D303: symbol BAR43 -> my_devices:BAR43
- J301: symbol RJ12 -> wfred_loconet_clock-rescue:RJ12
- K301: symbol CONN_3 -> wfred_loconet_clock-rescue:CONN_3
- Q301, Q302, Q303: symbol BC817-40 -> wfred_loconet_clock-rescue:BC817-40
- R301, R302, R303, R304, R305, R306, R307, R308, R309, R310: symbol R -> wfred_loconet_clock-rescue:R
- U301: symbol TC1240 -> my_devices:TC1240
Connections:
- wire segments 71 -> 93
Changed lines of the file:
@@
-EESchema Schematic File Version 2
-LIBS:power
-LIBS:device
-LIBS:transistors
-LIBS:conn
-LIBS:linear
-LIBS:regul
-LIBS:74xx
-LIBS:cmos4000
-LIBS:adc-dac
-LIBS:memory
-LIBS:xilinx
-LIBS:microcontrollers
-LIBS:dsp
-LIBS:microchip
-LIBS:analog_switches
-LIBS:motorola
-LIBS:texas
-LIBS:intel
-LIBS:audio
-LIBS:interface
-LIBS:digital-audio
-LIBS:philips
-LIBS:display
-LIBS:cypress
-LIBS:siliconi
-LIBS:opto
-LIBS:atmel
-LIBS:contrib
-LIBS:valves
-LIBS:my_devices
-LIBS:ESP8266
-LIBS:wfred_loconet_clock-cache
-EELAYER 25 0
+EESchema Schematic File Version 4
+EELAYER 30 0
 EELAYER END
 $Descr A4 11693 8268
@@
 $EndDescr
 $Comp
-L RJ12 J301
+L wfred_loconet_clock-rescue:RJ12 J301
 U 1 1 5920DD7A
 P 7350 2600
@@
 $EndComp
 $Comp
-L GND #PWR023
+L wfred_loconet_clock-rescue:GND #PWR023
 U 1 1 5920DF18
 P 6800 3300
@@
 	6900 2500 6800 2500
 Wire Wire Line
-	6800 2500 6800 3300
+	6800 2500 6800 2800
 Wire Wire Line
 	6900 2800 6800 2800
@@
 	7650 3100 7650 3200
 Wire Wire Line
-	6800 3200 7750 3200
+	6800 3200 7650 3200
 Connection ~ 6800 3200
 Wire Wire Line
@@
 	6200 2900 6300 2900
 Wire Wire Line
-	6200 2200 6200 2900
+	6200 2200 6200 2400
 Connection ~ 6200 2400
 $Comp
-L BAR43 D303
+L my_devices:BAR43 D303
 U 1 1 5920E30D
 P 6500 2900
@@
 $EndComp
 $Comp
-L BAR43 D302
+L my_devices:BAR43 D302
 U 1 1 5920E364
 P 6500 2400
@@
 $EndComp
 Wire Wire Line
-	5400 2600 6900 2600
+	5400 2600 5900 2600
 Wire Wire Line
 	6900 2700 6700 2700
@@
 Connection ~ 6700 2600
 $Comp
-L R R307
+L wfred_loconet_clock-rescue:R R307
 U 1 1 5920E41D
 P 5900 4150
@@
 $EndComp
 $Comp
-L R R308
+L wfred_loconet_clock-rescue:R R308
 U 1 1 5920E524
 P 5900 4850
@@
 $EndComp
 $Comp
-L C C302
+L wfred_loconet_clock-rescue:C C302
 U 1 1 5920E582
 P 6200 4800
@@
 $EndComp
 Wire Wire Line
-	5900 4400 5900 4600
+	5900 4400 5900 4500
 Wire Wire Line
 	5900 4500 6200 4500
@@
 Connection ~ 5900 4500
 $Comp
-L GND #PWR024
+L wfred_loconet_clock-rescue:GND #PWR024
 U 1 1 5920E62F
 P 6200 5100
@@
 	6200 5000 6200 5100
 $Comp
-L BC817-40 Q303
+L wfred_loconet_clock-rescue:BC817-40 Q303
 U 1 1 5920E776
 P 5800 5700
@@
 $EndComp
 $Comp
-L GND #PWR025
+L wfred_loconet_clock-rescue:GND #PWR025
 U 1 1 5920E813
 P 5900 6300
@@
 	5900 6300 5900 5900
 Wire Wire Line
-	5900 5100 5900 5500
-$Comp
-L R R306
+	5900 5100 5900 5200
+$Comp
+L wfred_loconet_clock-rescue:R R306
 U 1 1 5920E9B7
 P 5550 5200
@@
 $EndComp
 $Comp
-L R R304
+L wfred_loconet_clock-rescue:R R304
 U 1 1 5920EA5E
 P 4850 5200
@@
 $EndComp
 $Comp
-L R R305
+L wfred_loconet_clock-rescue:R R305
 U 1 1 5920EAAC
 P 5150 5700
@@
 $EndComp
 $Comp
-L R R302
+L wfred_loconet_clock-rescue:R R302
 U 1 1 5920EB49
 P 4200 5550
@@
 $EndComp
 $Comp
-L R R310
+L wfred_loconet_clock-rescue:R R310
 U 1 1 5920EBE7
 P 7650 5650
@@
 $EndComp
 $Comp
-L R R309
+L wfred_loconet_clock-rescue:R R309
 U 1 1 5920ECD0
 P 7650 4850
@@
 $EndComp
 $Comp
-L C C303
+L wfred_loconet_clock-rescue:C C303
 U 1 1 5920ED58
 P 7950 5650
@@
 $EndComp
 $Comp
-L C C301
+L wfred_loconet_clock-rescue:C C301
 U 1 1 5920EDE7
 P 5150 6000
@@
 $EndComp
 $Comp
-L BAR43 D301
+L my_devices:BAR43 D301
 U 1 1 5920EE82
 P 5200 4900
@@
 Connection ~ 5900 5200
 Wire Wire Line
-	5100 5200 5300 5200
+	5100 5200 5200 5200
 Wire Wire Line
 	5200 5100 5200 5200
 Connection ~ 5200 5200
 Wire Wire Line
-	3900 5200 4600 5200
+	3900 5200 4200 5200
 Wire Wire Line
 	4200 5200 4200 5300
 Wire Wire Line
-	5400 5700 5600 5700
+	5400 5700 5500 5700
 Wire Wire Line
 	5350 6000 5500 6000
@@
 Connection ~ 5500 5700
 Wire Wire Line
-	4700 5700 4900 5700
+	4700 5700 4800 5700
 Wire Wire Line
 	4950 6000 4800 6000
@@
 LN_TX
 $Comp
-L GND #PWR026
+L wfred_loconet_clock-rescue:GND #PWR026
 U 1 1 5920F1D7
 P 4200 6300
@@
 	4200 5800 4200 6300
 $Comp
-L VCC #PWR027
+L power:VCC #PWR027
 U 1 1 5920F266
 P 5200 4500
@@
 LN_RX0
 $Comp
-L GND #PWR028
+L wfred_loconet_clock-rescue:GND #PWR028
 U 1 1 5920F3BF
 P 7650 6300
@@
 $EndComp
 Wire Wire Line
-	7650 5900 7650 6300
+	7650 5900 7650 6000
 Wire Wire Line
 	7950 5850 7950 6000
@@
 Connection ~ 7650 6000
 Wire Wire Line
-	7650 5100 7650 5400
+	7650 5100 7650 5200
 Wire Wire Line
 	7950 5200 7950 5450
 Wire Wire Line
-	7150 5200 7950 5200
+	7150 5200 7650 5200
 Connection ~ 7650 5200
 $Comp
-L VCC #PWR029
+L power:VCC #PWR029
 U 1 1 5920F511
 P 7650 4500
@@
 LN_RX1
 $Comp
-L BC817-40 Q302
+L wfred_loconet_clock-rescue:BC817-40 Q302
 U 1 1 5920FF12
 P 4600 2200
@@
 $EndComp
 $Comp
-L BC817-40 Q301
+L wfred_loconet_clock-rescue:BC817-40 Q301
 U 1 1 59210062
 P 4300 2600
@@
 $EndComp
 $Comp
-L R R301
+L wfred_loconet_clock-rescue:R R301
 U 1 1 59210145
 P 4200 1850
@@
 $EndComp
 $Comp
-L R R303
+L wfred_loconet_clock-rescue:R R303
 U 1 1 5921022B
 P 4700 2950
@@
 $EndComp
 $Comp
-L CONN_3 K301
+L wfred_loconet_clock-rescue:CONN_3 K301
 U 1 1 59210360
 P 3750 1300
@@
 $EndComp
 Wire Wire Line
-	4100 1400 4700 1400
+	4100 1400 4200 1400
 Wire Wire Line
 	4200 1400 4200 1600
@@
 Connection ~ 4200 1400
 Wire Wire Line
-	4200 2100 4200 2400
+	4200 2100 4200 2200
 Wire Wire Line
 	4400 2200 4200 2200
 Connection ~ 4200 2200
 Wire Wire Line
-	4700 2400 4700 2700
+	4700 2400 4700 2600
 Wire Wire Line
 	4500 2600 4700 2600
@@
 	4200 2800 4200 3300
 Wire Wire Line
-	4200 3300 5400 3300
+	4200 3300 4700 3300
 Wire Wire Line
 	4700 3300 4700 3200
@@
 	4100 1200 4200 1200
 Wire Wire Line
-	4200 1000 4200 1300
-$Comp
-L TC1240 U301
+	4200 1000 4200 1200
+$Comp
+L my_devices:TC1240 U301
 U 1 1 5A1AB828
 P 2300 2400
@@
 $EndComp
 $Comp
-L C C304
+L wfred_loconet_clock-rescue:C C304
 U 1 1 5A1ABA44
 P 1300 2550
@@
 $EndComp
 $Comp
-L C C305
+L wfred_loconet_clock-rescue:C C305
 U 1 1 5A1ABAB1
 P 3200 2400
@@
 $EndComp
 $Comp
-L GND #PWR030
+L wfred_loconet_clock-rescue:GND #PWR030
 U 1 1 5A1ABBB5
 P 2300 3200
@@
 $EndComp
 $Comp
-L GND #PWR031
+L wfred_loconet_clock-rescue:GND #PWR031
 U 1 1 5A1ABBFB
 P 3200 3200
@@
 	3000 2700 3200 2700
 Wire Wire Line
-	3200 2600 3200 3200
+	3200 2600 3200 2700
 Connection ~ 3200 2700
 Wire Wire Line
@@
 	1500 2400 1600 2400
 $Comp
-L VCC #PWR032
+L power:VCC #PWR032
 U 1 1 5A1ABEC8
 P 1400 1950
@@
 	1400 2100 1600 2100
 $Comp
-L +5V #PWR033
+L power:+5V #PWR033
 U 1 1 5A1AC01A
 P 3200 1950
@@
 $EndComp
 Wire Wire Line
-	3200 1950 3200 2200
+	3200 1950 3200 2100
 Wire Wire Line
 	3000 2100 3200 2100
 Connection ~ 3200 2100
 $Comp
-L +5V #PWR034
+L power:+5V #PWR034
 U 1 1 5A1AC27E
 P 4200 1000
@@
 Connection ~ 4200 1200
 $Comp
-L +5V #PWR035
+L power:+5V #PWR035
 U 1 1 5A1AC467
 P 6200 2200
@@
 Wire Wire Line
 	6200 2400 6300 2400
+Wire Wire Line
+	6800 2800 6800 3200
+Wire Wire Line
+	6800 3200 6800 3300
+Wire Wire Line
+	7650 3200 7750 3200
+Wire Wire Line
+	6200 2400 6200 2900
+Wire Wire Line
+	6700 2600 6900 2600
+Wire Wire Line
+	5900 4500 5900 4600
+Wire Wire Line
+	5900 5200 5900 5500
+Wire Wire Line
+	5200 5200 5300 5200
+Wire Wire Line
+	5500 5700 5600 5700
+Wire Wire Line
+	4800 5700 4900 5700
+Wire Wire Line
+	4200 5200 4600 5200
+Wire Wire Line
+	7650 6000 7650 6300
+Wire Wire Line
+	7650 5200 7650 5400
+Wire Wire Line
+	7650 5200 7950 5200
+Wire Wire Line
+	4200 1400 4700 1400
+Wire Wire Line
+	4200 2200 4200 2400
+Wire Wire Line
+	4700 2600 4700 2700
+Wire Wire Line
+	4700 3300 5400 3300
+Wire Wire Line
+	5900 2600 6700 2600
+Wire Wire Line
+	3200 2700 3200 3200
+Wire Wire Line
+	3200 2100 3200 2200
+Wire Wire Line
+	4200 1200 4200 1300
 $EndSCHEMATC
