File: hardware/wfred-controller_rev2.sch (KiCad schematic (older format))
At the start: 10 parts, among them IC201 ATMEGA328P-A, P201 ISP, X201 myCRYSTAL

Commit message: Fixed up wfred_loconet_clock PCB...
...just in case someone actually wants to use it...
Parts:
- C201, C202, C203, C204, C205, C206: symbol C -> wfred_loconet_clock-rescue:C
- IC201: symbol ATMEGA328P-A -> wfred_loconet_clock-rescue:ATMEGA328P-A
- P201: symbol CONN_3X2 -> wfred_loconet_clock-rescue:CONN_3X2
- R201: symbol R -> wfred_loconet_clock-rescue:R
- X201: symbol myCRYSTAL -> my_devices:myCRYSTAL
Connections:
- wire segments 70 -> 89
Changed lines of the file:
@@
-EESchema Schematic File Version 2
-LIBS:power
-LIBS:device
-LIBS:transistors
-LIBS:conn
-LIBS:linear
-LIBS:regul
-LIBS:74xx
-LIBS:cmos4000
-LIBS:adc-dac
-LIBS:memory
-LIBS:xilinx
-LIBS:microcontrollers
-LIBS:dsp
-LIBS:microchip
-LIBS:analog_switches
-LIBS:motorola
-LIBS:texas
-LIBS:intel
-LIBS:audio
-LIBS:interface
-LIBS:digital-audio
-LIBS:philips
-LIBS:display
-LIBS:cypress
-LIBS:siliconi
-LIBS:opto
-LIBS:atmel
-LIBS:contrib
-LIBS:valves
-LIBS:my_devices
-LIBS:ESP8266
-LIBS:wfred_loconet_clock-cache
-EELAYER 25 0
+EESchema Schematic File Version 4
+EELAYER 30 0
 EELAYER END
 $Descr A4 11693 8268
@@
 $EndDescr
 $Comp
-L C C205
+L wfred_loconet_clock-rescue:C C205
 U 1 1 5920CFB6
 P 7700 3600
@@
 $EndComp
 $Comp
-L C C206
+L wfred_loconet_clock-rescue:C C206
 U 1 1 5920D023
 P 7700 4400
@@
 $EndComp
 $Comp
-L C C202
+L wfred_loconet_clock-rescue:C C202
 U 1 1 5920D0A7
 P 4400 2100
@@
 $EndComp
 $Comp
-L C C203
+L wfred_loconet_clock-rescue:C C203
 U 1 1 5920E33B
 P 4700 2100
@@
 $EndComp
 $Comp
-L C C204
+L wfred_loconet_clock-rescue:C C204
 U 1 1 5920E379
 P 5000 2100
@@
 $EndComp
 $Comp
-L C C201
+L wfred_loconet_clock-rescue:C C201
 U 1 1 5920E47C
 P 2100 4300
@@
 $EndComp
 $Comp
-L CONN_3X2 P201
+L wfred_loconet_clock-rescue:CONN_3X2 P201
 U 1 1 5920E592
 P 3500 2250
@@
 $EndComp
 $Comp
-L R R201
+L wfred_loconet_clock-rescue:R R201
 U 1 1 5920FD60
 P 3550 1700
@@
 MOSI
 $Comp
-L PWR_FLAG #FLG013
+L power:PWR_FLAG #FLG013
 U 1 1 59214642
 P 2100 3800
@@
 $EndComp
 $Comp
-L GND #PWR014
+L wfred_loconet_clock-rescue:GND #PWR014
 U 1 1 5920D54C
 P 8100 4600
@@
 $EndComp
 $Comp
-L GND #PWR015
+L wfred_loconet_clock-rescue:GND #PWR015
 U 1 1 5920D60E
 P 4400 2700
@@
 $EndComp
 $Comp
-L VCC #PWR016
+L power:VCC #PWR016
 U 1 1 5920D930
 P 4500 1500
@@
 $EndComp
 Wire Wire Line
-	6500 3600 7500 3600
+	6500 3600 7200 3600
 Wire Wire Line
 	7200 3600 7200 3700
@@
 	7200 4300 7200 4400
 Wire Wire Line
-	6500 4400 7500 4400
+	6500 4400 7200 4400
 Wire Wire Line
 	5000 1700 5000 1900
@@
 Connection ~ 4700 1700
 Wire Wire Line
-	4400 2300 4400 2700
-Wire Wire Line
-	4100 2500 5000 2500
+	4400 2300 4400 2500
+Wire Wire Line
+	4100 2500 4400 2500
 Wire Wire Line
 	4700 2500 4700 2300
@@
 	7900 3600 8100 3600
 Wire Wire Line
-	8100 3600 8100 4600
+	8100 3600 8100 4400
 Wire Wire Line
 	7900 4400 8100 4400
 Connection ~ 8100 4400
 Wire Wire Line
-	2100 3800 2100 4100
+	2100 3800 2100 3900
 Wire Wire Line
 	2100 4500 2100 4700
 Wire Wire Line
-	2900 2300 3100 2300
+	2900 2300 3000 2300
 Wire Wire Line
 	4100 2100 3900 2100
@@
 	4500 1700 4500 1500
 $Comp
-L ATMEGA328P-A IC201
+L wfred_loconet_clock-rescue:ATMEGA328P-A IC201
 U 1 1 592E0A20
 P 3900 4400
+AR Path="/592E0A20" Ref="IC201"  Part="1"
+AR Path="/5920C945/592E0A20" Ref="IC201"  Part="1"
 F 0 "IC201" H 3150 5650 40  0000 L BNN
 F 1 "ATMEGA328P-A" H 4300 3000 40  0000 L BNN
@@
 $EndComp
 Wire Wire Line
-	3800 1700 5000 1700
+	3800 1700 4100 1700
 Text GLabel 5100 5500 2    60   Input ~ 0
 LN_RX0
@@
 THIS_RXD
 $Comp
-L +BATT #PWR017
+L power:+BATT #PWR017
 U 1 1 592E1307
 P 2700 4200
@@
 	4900 3400 5350 3400
 Wire Wire Line
-	4900 3600 5350 3600
-Wire Wire Line
-	4900 3700 5350 3700
-Wire Wire Line
-	4900 3800 5350 3800
+	4900 3600 5000 3600
+Wire Wire Line
+	4900 3700 5100 3700
+Wire Wire Line
+	4900 3800 5200 3800
 Wire Wire Line
 	4900 4150 5100 4150
@@
 Connection ~ 3000 2300
 $Comp
-L VCC #PWR018
+L power:VCC #PWR018
 U 1 1 592F44B9
 P 2700 3100
@@
 $EndComp
 Wire Wire Line
-	2700 3100 2700 3600
+	2700 3100 2700 3300
 Wire Wire Line
 	2700 3300 3000 3300
@@
 Connection ~ 2700 3400
 $Comp
-L GND #PWR019
+L wfred_loconet_clock-rescue:GND #PWR019
 U 1 1 592F4690
 P 2100 4700
@@
 $EndComp
 $Comp
-L GND #PWR020
+L wfred_loconet_clock-rescue:GND #PWR020
 U 1 1 592F46BC
 P 2700 5900
@@
 $EndComp
 Wire Wire Line
-	2700 5400 2700 5900
+	2700 5400 2700 5500
 Wire Wire Line
 	2700 5600 3000 5600
@@
 ESTOP
 $Comp
-L myCRYSTAL X201
+L my_devices:myCRYSTAL X201
 U 1 1 5A171DD9
 P 7200 4000
@@
 $EndComp
 $Comp
-L GND #PWR021
+L wfred_loconet_clock-rescue:GND #PWR021
 U 1 1 5A171EC6
 P 7000 4600
@@
 $EndComp
 $Comp
-L GND #PWR022
+L wfred_loconet_clock-rescue:GND #PWR022
 U 1 1 5A171EEF
 P 6800 3800
@@
 Wire Wire Line
 	7000 4300 7000 4600
+Wire Wire Line
+	4700 1700 5000 1700
+Wire Wire Line
+	4400 2500 4400 2700
+Wire Wire Line
+	4400 2500 4700 2500
+Wire Wire Line
+	4700 2500 5000 2500
+Wire Wire Line
+	7200 3600 7500 3600
+Wire Wire Line
+	7200 4400 7500 4400
+Wire Wire Line
+	8100 4400 8100 4600
+Wire Wire Line
+	4100 1700 4400 1700
+Wire Wire Line
+	4400 1700 4500 1700
+Wire Wire Line
+	2100 3900 2100 4100
+Wire Wire Line
+	4500 1700 4700 1700
+Wire Wire Line
+	3000 2300 3100 2300
+Wire Wire Line
+	2700 3300 2700 3400
+Wire Wire Line
+	2700 3400 2700 3600
+Wire Wire Line
+	2700 5600 2700 5900
+Wire Wire Line
+	2700 5500 2700 5600
+Wire Wire Line
+	5000 3600 5350 3600
+Wire Wire Line
+	5100 3700 5350 3700
+Wire Wire Line
+	5200 3800 5350 3800
 $EndSCHEMATC
