File: hardware/wfred-wifi.sch (KiCad schematic (older format))
At the start: 11 parts, among them K401 UART_ESP, K402 UART_AVR, P401 ESP_BOOTLOAD, U401 ESP-12E

Commit message: Fixed up wfred_loconet_clock PCB...
...just in case someone actually wants to use it...
Parts:
- C401, C402: symbol C -> wfred_loconet_clock-rescue:C
- K401, K402: symbol CONN_3 -> wfred_loconet_clock-rescue:CONN_3
- P401: symbol CONN_2 -> wfred_loconet_clock-rescue:CONN_2
- R401, R402, R403, R404, R405: symbol R -> wfred_loconet_clock-rescue:R
- U401: symbol ESP-12E -> wfred_loconet_clock-rescue:ESP-12E-ESP8266
Changed lines of the file:
@@
-EESchema Schematic File Version 2
-LIBS:power
-LIBS:device
-LIBS:transistors
-LIBS:conn
-LIBS:linear
-LIBS:regul
-LIBS:74xx
-LIBS:cmos4000
-LIBS:adc-dac
-LIBS:memory
-LIBS:xilinx
-LIBS:microcontrollers
-LIBS:dsp
-LIBS:microchip
-LIBS:analog_switches
-LIBS:motorola
-LIBS:texas
-LIBS:intel
-LIBS:audio
-LIBS:interface
-LIBS:digital-audio
-LIBS:philips
-LIBS:display
-LIBS:cypress
-LIBS:siliconi
-LIBS:opto
-LIBS:atmel
-LIBS:contrib
-LIBS:valves
-LIBS:my_devices
-LIBS:ESP8266
-LIBS:wfred_loconet_clock-cache
-EELAYER 25 0
+EESchema Schematic File Version 4
+EELAYER 30 0
 EELAYER END
 $Descr A4 11693 8268
@@
 $EndDescr
 $Comp
-L ESP-12E U401
+L wfred_loconet_clock-rescue:ESP-12E-ESP8266 U401
 U 1 1 5A11AA62
 P 4300 2600
@@
 $EndComp
 $Comp
-L +BATT #PWR036
+L power:+BATT #PWR036
 U 1 1 5A11AB98
 P 2500 1500
@@
 	2500 1500 2500 1800
 $Comp
-L R R401
+L wfred_loconet_clock-rescue:R R401
 U 1 1 5A11AE00
 P 2500 2050
@@
 $EndComp
 $Comp
-L R R402
+L wfred_loconet_clock-rescue:R R402
 U 1 1 5A11AE49
 P 2500 2750
@@
 $EndComp
 Wire Wire Line
-	2500 2300 2500 2500
+	2500 2300 2500 2400
 Wire Wire Line
 	3400 2400 2500 2400
 Connection ~ 2500 2400
 $Comp
-L GND #PWR037
+L wfred_loconet_clock-rescue:GND #PWR037
 U 1 1 5A11B098
 P 2500 3700
@@
 NoConn ~ 4550 3500
 $Comp
-L VCC #PWR038
+L power:VCC #PWR038
 U 1 1 5A11E004
 P 2700 1500
@@
 $EndComp
 Wire Wire Line
-	2700 1500 2700 3000
+	2700 1500 2700 2300
 Wire Wire Line
 	2700 2300 3400 2300
@@
 Connection ~ 2700 2500
 $Comp
-L GND #PWR039
+L wfred_loconet_clock-rescue:GND #PWR039
 U 1 1 5A11E30D
 P 6700 3700
@@
 $EndComp
 Wire Wire Line
-	6700 2500 6700 3700
+	6700 2500 6700 2900
 Wire Wire Line
 	6700 3000 5200 3000
 Connection ~ 6700 3000
 $Comp
-L VCC #PWR040
+L power:VCC #PWR040
 U 1 1 5A11E4AA
 P 6300 1550
@@
 	5200 2400 6750 2400
 $Comp
-L CONN_3 K401
+L wfred_loconet_clock-rescue:CONN_3 K401
 U 1 1 5A11EE74
 P 7100 2400
@@
 THIS_TXD
 $Comp
-L CONN_2 P401
+L wfred_loconet_clock-rescue:CONN_2 P401
 U 1 1 5A11F720
 P 7100 2800
@@
 $EndComp
 Wire Wire Line
-	5200 2700 6750 2700
-$Comp
-L GND #PWR041
+	5200 2700 6100 2700
+$Comp
+L wfred_loconet_clock-rescue:GND #PWR041
 U 1 1 5A11FC27
 P 7850 2500
@@
 $EndComp
 $Comp
-L R R403
+L wfred_loconet_clock-rescue:R R403
 U 1 1 5A11FF91
 P 6100 1950
@@
 $EndComp
 $Comp
-L R R404
+L wfred_loconet_clock-rescue:R R404
 U 1 1 5A11FFE4
 P 6100 3350
@@
 $EndComp
 $Comp
-L R R405
+L wfred_loconet_clock-rescue:R R405
 U 1 1 5A120047
 P 6300 1950
@@
 	5200 2900 6100 2900
 $Comp
-L CONN_3 K402
+L wfred_loconet_clock-rescue:CONN_3 K402
 U 1 1 5A11F053
 P 7350 2300
@@
 	6100 1700 6100 1600
 Wire Wire Line
-	6300 1550 6300 1700
+	6300 1550 6300 1600
 Connection ~ 6300 1600
 Wire Wire Line
 	6100 2900 6100 3100
 $Comp
-L GND #PWR042
+L wfred_loconet_clock-rescue:GND #PWR042
 U 1 1 5A120E87
 P 6100 3700
@@
 	5400 2600 5200 2600
 $Comp
-L C C401
+L wfred_loconet_clock-rescue:C C401
 U 1 1 5A127BCA
 P 1400 2400
@@
 $EndComp
 $Comp
-L VCC #PWR043
+L power:VCC #PWR043
 U 1 1 5A127C0E
 P 1400 1800
@@
 $EndComp
 Wire Wire Line
-	1400 1800 1400 2200
-$Comp
-L GND #PWR044
+	1400 1800 1400 2000
+$Comp
+L wfred_loconet_clock-rescue:GND #PWR044
 U 1 1 5A127CDB
 P 1400 2900
@@
 $EndComp
 Wire Wire Line
-	1400 2900 1400 2600
-$Comp
-L C C402
+	1400 2900 1400 2800
+$Comp
+L wfred_loconet_clock-rescue:C C402
 U 1 1 5A199174
 P 1700 2400
@@
 	1700 2800 1400 2800
 Connection ~ 1400 2800
+Wire Wire Line
+	2500 2400 2500 2500
+Wire Wire Line
+	2700 2300 2700 2500
+Wire Wire Line
+	2700 2500 2700 3000
+Wire Wire Line
+	6700 3000 6700 3700
+Wire Wire Line
+	6100 2700 6750 2700
+Wire Wire Line
+	6300 1600 6300 1700
+Wire Wire Line
+	6700 2900 6700 3000
+Wire Wire Line
+	1400 2000 1400 2200
+Wire Wire Line
+	1400 2800 1400 2600
 $EndSCHEMATC
