File: hardware/wfred_loconet_clock.sch (KiCad schematic (older format))
At the start: 8 parts, among them U101 L6920D

Commit message: Fixed up wfred_loconet_clock PCB...
...just in case someone actually wants to use it...
Parts:
- B101: symbol BATT_HOLDER -> my_devices:BATT_HOLDER
- C101, C102, C103, C104, C105: symbol C -> wfred_loconet_clock-rescue:C
- L101: symbol INDUCTOR -> wfred_loconet_clock-rescue:INDUCTOR
- U101: symbol L6920D -> my_devices:L6920D
Changed lines of the file:
@@
-EESchema Schematic File Version 2
-LIBS:power
-LIBS:device
-LIBS:transistors
-LIBS:conn
-LIBS:linear
-LIBS:regul
-LIBS:74xx
-LIBS:cmos4000
-LIBS:adc-dac
-LIBS:memory
-LIBS:xilinx
-LIBS:microcontrollers
-LIBS:dsp
-LIBS:microchip
-LIBS:analog_switches
-LIBS:motorola
-LIBS:texas
-LIBS:intel
-LIBS:audio
-LIBS:interface
-LIBS:digital-audio
-LIBS:philips
-LIBS:display
-LIBS:cypress
-LIBS:siliconi
-LIBS:opto
-LIBS:atmel
-LIBS:contrib
-LIBS:valves
-LIBS:my_devices
-LIBS:ESP8266
-LIBS:wfred_loconet_clock-cache
-EELAYER 25 0
+EESchema Schematic File Version 4
+EELAYER 30 0
 EELAYER END
 $Descr A4 11693 8268
@@
 $EndDescr
 Wire Wire Line
-	2450 2450 2450 2700
-Wire Wire Line
-	900  2600 2450 2600
-Wire Wire Line
-	2150 2400 2150 2700
+	2450 2450 2450 2600
+Wire Wire Line
+	900  2600 2150 2600
+Wire Wire Line
+	2150 2400 2150 2600
 Connection ~ 2150 2600
 Wire Wire Line
 	1500 2800 1850 2800
 Wire Wire Line
-	1850 2450 1850 3300
+	1850 2450 1850 2800
 Wire Wire Line
 	2150 3100 2150 3300
@@
 	3300 3100 3300 3300
 Wire Wire Line
-	5200 2000 5200 2800
-Wire Wire Line
-	5000 2200 6600 2200
+	5200 2000 5200 2200
+Wire Wire Line
+	5000 2200 5200 2200
 Wire Wire Line
 	5200 2800 5000 2800
@@
 Connection ~ 5500 2200
 $Comp
-L C C101
+L wfred_loconet_clock-rescue:C C101
 U 1 1 5920B38E
 P 2150 2900
@@
 $EndComp
 $Comp
-L GND #PWR01
+L wfred_loconet_clock-rescue:GND #PWR01
 U 1 1 5920B390
 P 2150 3300
@@
 $EndComp
 $Comp
-L GND #PWR02
+L wfred_loconet_clock-rescue:GND #PWR02
 U 1 1 5920B391
 P 1850 3300
@@
 $EndComp
 $Comp
-L GND #PWR03
+L wfred_loconet_clock-rescue:GND #PWR03
 U 1 1 5920B392
 P 2450 3300
@@
 $EndComp
 $Comp
-L +BATT #PWR04
+L power:+BATT #PWR04
 U 1 1 5920B394
 P 2150 2400
@@
 $EndComp
 $Comp
-L INDUCTOR L101
+L wfred_loconet_clock-rescue:INDUCTOR L101
 U 1 1 5920B395
 P 4300 1400
@@
 $EndComp
 $Comp
-L +BATT #PWR05
+L power:+BATT #PWR05
 U 1 1 5920B396
 P 4300 900
@@
 NoConn ~ 3600 2200
 $Comp
-L C C103
+L wfred_loconet_clock-rescue:C C103
 U 1 1 5920B397
 P 3300 2900
@@
 $EndComp
 $Comp
-L GND #PWR06
+L wfred_loconet_clock-rescue:GND #PWR06
 U 1 1 5920B398
 P 3300 3300
@@
 $EndComp
 $Comp
-L GND #PWR07
+L wfred_loconet_clock-rescue:GND #PWR07
 U 1 1 5920B399
 P 3500 3300
@@
 NoConn ~ 5000 2500
 $Comp
-L VCC #PWR08
+L power:VCC #PWR08
 U 1 1 5920B39A
 P 5200 2000
@@
 $EndComp
 $Comp
-L GND #PWR09
+L wfred_loconet_clock-rescue:GND #PWR09
 U 1 1 5920B39D
 P 6300 3300
@@
 $EndComp
 $Comp
-L GND #PWR010
+L wfred_loconet_clock-rescue:GND #PWR010
 U 1 1 5920B39E
 P 6600 3300
@@
 $EndSheet
 $Comp
-L C C102
+L wfred_loconet_clock-rescue:C C102
 U 1 1 59210DD0
 P 2450 2900
@@
 $EndComp
 $Comp
-L C C104
+L wfred_loconet_clock-rescue:C C104
 U 1 1 59210E13
 P 6300 2600
@@
 $EndComp
 $Comp
-L C C105
+L wfred_loconet_clock-rescue:C C105
 U 1 1 59210E8B
 P 6600 2600
@@
 $EndComp
 $Comp
-L PWR_FLAG #FLG011
+L power:PWR_FLAG #FLG011
 U 1 1 59214833
 P 2450 2450
@@
 Connection ~ 2450 2600
 $Comp
-L PWR_FLAG #FLG012
+L power:PWR_FLAG #FLG012
 U 1 1 59214BB2
 P 1850 2450
@@
 Connection ~ 1850 2800
 $Comp
-L L6920D U101
+L my_devices:L6920D U101
 U 1 1 5920B393
 P 4300 2500
@@
 	1500 3700 1500 2800
 $Comp
-L BATT_HOLDER B101
+L my_devices:BATT_HOLDER B101
 U 1 1 5A14A6C1
 P 1200 4900
@@
 	0    1    1    0
 $EndComp
+Wire Wire Line
+	2150 2600 2450 2600
+Wire Wire Line
+	2150 2600 2150 2700
+Wire Wire Line
+	5200 2200 5200 2800
+Wire Wire Line
+	5200 2200 5500 2200
+Wire Wire Line
+	6300 2200 6600 2200
+Wire Wire Line
+	5500 2200 6300 2200
+Wire Wire Line
+	2450 2600 2450 2700
+Wire Wire Line
+	1850 2800 1850 3300
 $EndSCHEMATC
